Commit message: spawned robot in custom gazebo world

File: my_robot_description/urdf/mobile_base.xacro (robot description, xacro)
@@ -100,5 +100,5 @@
         <parent link="base_link"/>
         <child link="base footprint"/>
-        <origin xyz="0.0 0.0 ${-base_height / 4.0}" rpy="0.0 0.0 0.0"/>
+        <origin xyz="0.0 0.0 ${base_height / 4.0}" rpy="0.0 0.0 0.0"/>
     </joint>
 </robot>
